File: LM3909.kicad_pcb (KiCad board)
At the start: 2 copper layers, 17 parts, among them Q1 BC847, Q2A1 BC807, Q2B1 BC807, Q3 BC847, Q4 BC847

Commit message: pretty dang small
Parts:
- moved R8 1.27 mm to (137.8, 110.5)
- moved Q2B1 1.27 mm to (136.5, 118.1)
- moved Q3 1.27 mm to (134.6, 109.2)
Routing:
- net Net-(BT1-Pad1): track 40.2 -> 38.4 mm
- net Net-(C1-Pad1): track 12.7 -> 10.9 mm
- net Net-(BT1-Pad2): track 30.2 -> 28.9 mm
- net Net-(Q1-Pad3): track 6.55 -> 7.26 mm
Changed lines of the file:
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@@
   )
   (module Resistors_SMD:R_0805 (layer F.Cu)
-    (at 139.065 110.49 90)
+    (at 137.795 110.49 90)
     (descr "Resistor SMD 0805, reflow soldering, Vishay (see dcrcw.pdf)")
     (tags "resistor 0805")
@@
   )
   (module TO_SOT_Packages_SMD:SOT-23 (layer F.Cu)
-    (at 136.525 119.38)
+    (at 136.525 118.11)
     (descr "SOT-23, Standard")
     (tags SOT-23)
@@
   )
   (module TO_SOT_Packages_SMD:SOT-23 (layer F.Cu)
-    (at 135.89 109.22 180)
+    (at 134.62 109.22 180)
     (descr "SOT-23, Standard")
     (tags SOT-23)
@@
     )
   )
-  (segment (start 127.955 113.03) (end 127.955 110.81) (width 0.25) (layer F.Cu) (net 1))
-  (segment (start 134.255 109.855) (end 134.89 109.22) (width 0.25) (layer F.Cu) (net 1))
-  (segment (start 128.91 109.855) (end 134.255 109.855) (width 0.25) (layer F.Cu) (net 1))
-  (segment (start 127.955 110.81) (end 128.91 109.855) (width 0.25) (layer F.Cu) (net 1))
-  (segment (start 127.955 113.03) (end 127.365 113.03) (width 0.25) (layer F.Cu) (net 1))
-  (segment (start 127.365 113.03) (end 125.73 111.395) (width 0.25) (layer F.Cu) (net 1))
+  (segment (start 127.955 113.03) (end 127.955 112.62) (width 0.25) (layer F.Cu) (net 1))
+  (segment (start 127.955 112.62) (end 126.73 111.395) (width 0.25) (layer F.Cu) (net 1))
+  (segment (start 125.73 111.395) (end 126.73 111.395) (width 0.25) (layer F.Cu) (net 1))
+  (segment (start 132.985 109.855) (end 133.62 109.22) (width 0.25) (layer F.Cu) (net 1))
+  (segment (start 128.27 109.855) (end 132.985 109.855) (width 0.25) (layer F.Cu) (net 1))
+  (segment (start 126.73 111.395) (end 128.27 109.855) (width 0.25) (layer F.Cu) (net 1))
   (segment (start 125.73 113.395) (end 123.29 113.395) (width 0.25) (layer F.Cu) (net 2))
   (segment (start 123.29 113.395) (end 123.19 113.495) (width 0.25) (layer F.Cu) (net 2))
@@
   (segment (start 125.63 113.495) (end 125.73 113.395) (width 0.25) (layer F.Cu) (net 2))
   (segment (start 125.73 113.395) (end 125.63 113.395) (width 0.25) (layer F.Cu) (net 2))
-  (segment (start 123.19 111.295) (end 123.19 109.535) (width 0.25) (layer F.Cu) (net 3) (status C00000))
-  (segment (start 123.19 109.535) (end 123.505 109.22) (width 0.25) (layer F.Cu) (net 3) (status C00000))
+  (segment (start 123.19 111.295) (end 123.19 109.535) (width 0.25) (layer F.Cu) (net 3))
+  (segment (start 123.19 109.535) (end 123.505 109.22) (width 0.25) (layer F.Cu) (net 3))
   (segment (start 127.905 117.79) (end 125.73 117.79) (width 0.25) (layer F.Cu) (net 4))
-  (segment (start 135.525 118.43) (end 134.035 118.43) (width 0.25) (layer F.Cu) (net 5))
+  (segment (start 133.715 118.11) (end 134.575 118.11) (width 0.25) (layer F.Cu) (net 5))
+  (segment (start 134.575 118.11) (end 135.525 117.16) (width 0.25) (layer F.Cu) (net 5))
   (segment (start 134.035 118.43) (end 133.715 118.11) (width 0.25) (layer F.Cu) (net 5))
   (segment (start 129.905 116.84) (end 131.395 116.84) (width 0.25) (layer F.Cu) (net 5))
@@
   (segment (start 127.905 115.89) (end 131.44 115.89) (width 0.25) (layer F.Cu) (net 6))
   (segment (start 131.44 115.89) (end 132.08 115.25) (width 0.25) (layer F.Cu) (net 6))
-  (segment (start 121.605 109.22) (end 121.605 108.9) (width 0.25) (layer F.Cu) (net 7) (status C00000))
-  (segment (start 121.605 108.9) (end 122.555 107.95) (width 0.25) (layer F.Cu) (net 7) (status 400000))
-  (segment (start 128.585 107.95) (end 129.54 108.905) (width 0.25) (layer F.Cu) (net 7) (status 800000))
+  (segment (start 135.525 119.06) (end 135.575 119.06) (width 0.25) (layer F.Cu) (net 7))
+  (segment (start 135.575 119.06) (end 136.525 118.11) (width 0.25) (layer F.Cu) (net 7))
+  (segment (start 136.525 116.57) (end 137.795 115.3) (width 0.25) (layer F.Cu) (net 7))
+  (segment (start 136.525 118.11) (end 136.525 116.57) (width 0.25) (layer F.Cu) (net 7))
+  (segment (start 131.715 119.06) (end 135.525 119.06) (width 0.25) (layer F.Cu) (net 7))
+  (segment (start 121.605 109.22) (end 121.605 108.9) (width 0.25) (layer F.Cu) (net 7))
+  (segment (start 121.605 108.9) (end 122.555 107.95) (width 0.25) (layer F.Cu) (net 7))
+  (segment (start 128.585 107.95) (end 129.54 108.905) (width 0.25) (layer F.Cu) (net 7))
   (segment (start 122.555 107.95) (end 128.585 107.95) (width 0.25) (layer F.Cu) (net 7))
-  (segment (start 121.92 109.535) (end 121.92 110.49) (width 0.25) (layer F.Cu) (net 7) (status 400000))
+  (segment (start 121.92 109.535) (end 121.92 110.49) (width 0.25) (layer F.Cu) (net 7))
   (segment (start 124.78 119.06) (end 123.825 120.015) (width 0.25) (layer F.Cu) (net 7))
   (segment (start 123.825 120.015) (end 122.555 120.015) (width 0.25) (layer F.Cu) (net 7))
@@
   (segment (start 121.92 119.38) (end 121.92 110.49) (width 0.25) (layer F.Cu) (net 7))
   (segment (start 124.78 119.06) (end 131.715 119.06) (width 0.25) (layer F.Cu) (net 7))
-  (segment (start 121.92 109.535) (end 121.605 109.22) (width 0.25) (layer F.Cu) (net 7) (status C00000))
-  (segment (start 135.525 120.33) (end 135.575 120.33) (width 0.25) (layer F.Cu) (net 7))
-  (segment (start 135.575 120.33) (end 136.525 119.38) (width 0.25) (layer F.Cu) (net 7))
-  (segment (start 136.525 116.57) (end 137.795 115.3) (width 0.25) (layer F.Cu) (net 7))
-  (segment (start 136.525 119.38) (end 136.525 116.57) (width 0.25) (layer F.Cu) (net 7))
-  (segment (start 135.525 120.33) (end 132.985 120.33) (width 0.25) (layer F.Cu) (net 7))
-  (segment (start 132.985 120.33) (end 131.715 119.06) (width 0.25) (layer F.Cu) (net 7))
+  (segment (start 121.92 109.535) (end 121.605 109.22) (width 0.25) (layer F.Cu) (net 7))
   (segment (start 131.715 119.06) (end 131.715 119.11) (width 0.25) (layer F.Cu) (net 7))
-  (segment (start 137.525 119.38) (end 139.38 119.38) (width 0.25) (layer F.Cu) (net 8))
-  (segment (start 139.38 119.38) (end 139.7 119.06) (width 0.25) (layer F.Cu) (net 8))
-  (segment (start 120.97 118.745) (end 120.97 110.81) (width 0.25) (layer F.Cu) (net 9) (status 400000))
-  (segment (start 135.935 107.315) (end 136.89 108.27) (width 0.25) (layer F.Cu) (net 9) (status 800000))
-  (segment (start 121.92 107.315) (end 135.935 107.315) (width 0.25) (layer F.Cu) (net 9))
-  (segment (start 120.65 108.585) (end 121.92 107.315) (width 0.25) (layer F.Cu) (net 9))
-  (segment (start 120.65 110.49) (end 120.65 108.585) (width 0.25) (layer F.Cu) (net 9))
-  (segment (start 120.97 110.81) (end 120.65 110.49) (width 0.25) (layer F.Cu) (net 9))
-  (segment (start 139.065 109.54) (end 138.16 109.54) (width 0.25) (layer F.Cu) (net 9))
-  (segment (start 138.16 109.54) (end 136.89 108.27) (width 0.25) (layer F.Cu) (net 9))
+  (segment (start 137.525 118.11) (end 138.75 118.11) (width 0.25) (layer F.Cu) (net 8))
+  (segment (start 138.75 118.11) (end 139.7 119.06) (width 0.25) (layer F.Cu) (net 8))
+  (segment (start 135.62 108.27) (end 130.495 108.27) (width 0.25) (layer F.Cu) (net 9))
+  (segment (start 120.65 108.585) (end 120.65 118.425) (width 0.25) (layer F.Cu) (net 9))
+  (segment (start 121.92 107.315) (end 120.65 108.585) (width 0.25) (layer F.Cu) (net 9))
+  (segment (start 129.54 107.315) (end 121.92 107.315) (width 0.25) (layer F.Cu) (net 9))
+  (segment (start 130.495 108.27) (end 129.54 107.315) (width 0.25) (layer F.Cu) (net 9))
+  (segment (start 120.65 118.425) (end 120.97 118.745) (width 0.25) (layer F.Cu) (net 9))
+  (segment (start 137.795 109.54) (end 136.89 109.54) (width 0.25) (layer F.Cu) (net 9))
+  (segment (start 136.89 109.54) (end 135.62 108.27) (width 0.25) (layer F.Cu) (net 9))
+  (segment (start 136.845 113.3) (end 136.845 112.39) (width 0.25) (layer F.Cu) (net 10))
+  (segment (start 136.845 112.39) (end 137.795 111.44) (width 0.25) (layer F.Cu) (net 10))
   (segment (start 136.845 113.3) (end 137.205 113.3) (width 0.25) (layer F.Cu) (net 10))
-  (segment (start 137.205 113.3) (end 139.065 111.44) (width 0.25) (layer F.Cu) (net 10))
   (segment (start 134.62 113.35) (end 136.795 113.35) (width 0.25) (layer F.Cu) (net 10))
   (segment (start 136.795 113.35) (end 136.845 113.3) (width 0.25) (layer F.Cu) (net 10))
@@
   (segment (start 122.87 118.745) (end 122.87 117.475) (width 0.25) (layer F.Cu) (net 12))
   (segment (start 122.87 117.475) (end 123.19 117.155) (width 0.25) (layer F.Cu) (net 12))
-  (segment (start 136.89 110.17) (end 138.11 110.17) (width 0.25) (layer F.Cu) (net 13))
+  (segment (start 139.7 113.03) (end 139.7 111.76) (width 0.25) (layer F.Cu) (net 13))
+  (segment (start 138.43 110.49) (end 135.94 110.49) (width 0.25) (layer F.Cu) (net 13))
+  (segment (start 139.7 111.76) (end 138.43 110.49) (width 0.25) (layer F.Cu) (net 13))
+  (segment (start 135.94 110.49) (end 135.62 110.17) (width 0.25) (layer F.Cu) (net 13))
   (segment (start 139.7 113.03) (end 139.7 117.16) (width 0.25) (layer F.Cu) (net 13))
-  (segment (start 140.335 112.395) (end 139.7 113.03) (width 0.25) (layer F.Cu) (net 13))
-  (segment (start 140.335 111.125) (end 140.335 112.395) (width 0.25) (layer F.Cu) (net 13))
-  (segment (start 139.7 110.49) (end 140.335 111.125) (width 0.25) (layer F.Cu) (net 13))
-  (segment (start 138.43 110.49) (end 139.7 110.49) (width 0.25) (layer F.Cu) (net 13))
-  (segment (start 138.11 110.17) (end 138.43 110.49) (width 0.25) (layer F.Cu) (net 13))
+  (segment (start 139.7 113.03) (end 139.7 113.03) (width 0.25) (layer F.Cu) (net 13))
 )

Commit message: add through hole pin footprint
Parts:
- added J1: Conn_01x04, Pin_Headers:Pin_Header_Straight_1x04_Pitch2.54mm, F.Cu at (127.0, 127.0)
- added J2: Conn_01x04, Pin_Headers:Pin_Header_Straight_1x04_Pitch2.54mm, F.Cu at (134.6, 101.6)
Changed lines of the file:
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@@
 (kicad_pcb (version 4) (host pcbnew 4.0.7)
   (general
-    (links 26)
-    (no_connects 0)
+    (links 32)
+    (no_connects 6)
     (area 0 0 0 0)
     (thickness 1.6)
@@
     (tracks 74)
     (zones 0)
-    (modules 17)
-    (nets 14)
+    (modules 19)
+    (nets 16)
   )
   (page A4)
@@
   (net 10 "Net-(Q4-Pad2)")
   (net 11 "Net-(Q4-Pad1)")
-  (net 12 "Net-(R2-Pad2)")
-  (net 13 "Net-(Q3-Pad1)")
+  (net 12 "Net-(Q3-Pad1)")
+  (net 13 "Net-(J1-Pad1)")
+  (net 14 "Net-(J1-Pad3)")
+  (net 15 "Net-(J2-Pad3)")
   (net_class Default "This is the default net class."
     (clearance 0.2)
@@
     (add_net "Net-(C1-Pad2)")
     (add_net "Net-(D1-Pad2)")
+    (add_net "Net-(J1-Pad1)")
+    (add_net "Net-(J1-Pad3)")
+    (add_net "Net-(J2-Pad3)")
     (add_net "Net-(Q1-Pad1)")
     (add_net "Net-(Q1-Pad2)")
@@
     (add_net "Net-(Q4-Pad1)")
     (add_net "Net-(Q4-Pad2)")
-    (add_net "Net-(R2-Pad2)")
   )
   (module Resistors_SMD:R_0805 (layer F.Cu)
@@
       (net 2 "Net-(C1-Pad2)"))
     (pad 2 smd rect (at 0.95 0 270) (size 0.7 1.3) (layers F.Cu F.Paste F.Mask)
-      (net 12 "Net-(R2-Pad2)"))
+      (net 13 "Net-(J1-Pad1)"))
     (model ${KISYS3DMOD}/Resistors_SMD.3dshapes/R_0805.wrl
       (at (xyz 0 0 0))
@@
     (fp_line (start 1.55 0.9) (end -1.55 0.9) (layer F.CrtYd) (width 0.05))
     (pad 1 smd rect (at -0.95 0 180) (size 0.7 1.3) (layers F.Cu F.Paste F.Mask)
-      (net 12 "Net-(R2-Pad2)"))
+      (net 13 "Net-(J1-Pad1)"))
     (pad 2 smd rect (at 0.95 0 180) (size 0.7 1.3) (layers F.Cu F.Paste F.Mask)
       (net 9 "Net-(BT1-Pad2)"))
@@
     (fp_line (start 0.76 1.58) (end -0.7 1.58) (layer F.SilkS) (width 0.12))
     (pad 1 smd rect (at -1 -0.95 180) (size 0.9 0.8) (layers F.Cu F.Paste F.Mask)
-      (net 13 "Net-(Q3-Pad1)"))
+      (net 12 "Net-(Q3-Pad1)"))
     (pad 2 smd rect (at -1 0.95 180) (size 0.9 0.8) (layers F.Cu F.Paste F.Mask)
       (net 9 "Net-(BT1-Pad2)"))
@@
       (net 8 "Net-(Q2B1-Pad3)"))
     (pad 2 smd rect (at 0.95 0 90) (size 0.7 1.3) (layers F.Cu F.Paste F.Mask)
-      (net 13 "Net-(Q3-Pad1)"))
-    (model ${KISYS3DMOD}/Resistors_SMD.3dshapes/R_0805.wrl
+      (net 12 "Net-(Q3-Pad1)"))
+    (model ${KISYS3DMOD}/Resistors_SMD.3dshapes/R_0805.wrl
+      (at (xyz 0 0 0))
+      (scale (xyz 1 1 1))
+      (rotate (xyz 0 0 0))
+    )
+  )
+  (module Pin_Headers:Pin_Header_Straight_1x04_Pitch2.54mm (layer F.Cu)
+    (at 127 127 90)
+    (descr "Through hole straight pin header, 1x04, 2.54mm pitch, single row")
+    (tags "Through hole pin header THT 1x04 2.54mm single row")
+    (fp_text reference J1 (at 0 -2.33 90) (layer F.SilkS)
+      (effects (font (size 1 1) (thickness 0.15)))
+    )
+    (fp_text value Conn_01x04 (at 0 9.95 90) (layer F.Fab)
+      (effects (font (size 1 1) (thickness 0.15)))
+    )
+    (fp_line (start -0.635 -1.27) (end 1.27 -1.27) (layer F.Fab) (width 0.1))
+    (fp_line (start 1.27 -1.27) (end 1.27 8.89) (layer F.Fab) (width 0.1))
+    (fp_line (start 1.27 8.89) (end -1.27 8.89) (layer F.Fab) (width 0.1))
+    (fp_line (start -1.27 8.89) (end -1.27 -0.635) (layer F.Fab) (width 0.1))
+    (fp_line (start -1.27 -0.635) (end -0.635 -1.27) (layer F.Fab) (width 0.1))
+    (fp_line (start -1.33 8.95) (end 1.33 8.95) (layer F.SilkS) (width 0.12))
+    (fp_line (start -1.33 1.27) (end -1.33 8.95) (layer F.SilkS) (width 0.12))
+    (fp_line (start 1.33 1.27) (end 1.33 8.95) (layer F.SilkS) (width 0.12))
+    (fp_line (start -1.33 1.27) (end 1.33 1.27) (layer F.SilkS) (width 0.12))
+    (fp_line (start -1.33 0) (end -1.33 -1.33) (layer F.SilkS) (width 0.12))
+    (fp_line (start -1.33 -1.33) (end 0 -1.33) (layer F.SilkS) (width 0.12))
+    (fp_line (start -1.8 -1.8) (end -1.8 9.4) (layer F.CrtYd) (width 0.05))
+    (fp_line (start -1.8 9.4) (end 1.8 9.4) (layer F.CrtYd) (width 0.05))
+    (fp_line (start 1.8 9.4) (end 1.8 -1.8) (layer F.CrtYd) (width 0.05))
+    (fp_line (start 1.8 -1.8) (end -1.8 -1.8) (layer F.CrtYd) (width 0.05))
+    (fp_text user %R (at 0 3.81 180) (layer F.Fab)
+      (effects (font (size 1 1) (thickness 0.15)))
+    )
+    (pad 1 thru_hole rect (at 0 0 90) (size 1.7 1.7) (drill 1) (layers *.Cu *.Mask)
+      (net 13 "Net-(J1-Pad1)"))
+    (pad 2 thru_hole oval (at 0 2.54 90) (size 1.7 1.7) (drill 1) (layers *.Cu *.Mask)
+      (net 1 "Net-(C1-Pad1)"))
+    (pad 3 thru_hole oval (at 0 5.08 90) (size 1.7 1.7) (drill 1) (layers *.Cu *.Mask)
+      (net 14 "Net-(J1-Pad3)"))
+    (pad 4 thru_hole oval (at 0 7.62 90) (size 1.7 1.7) (drill 1) (layers *.Cu *.Mask)
+      (net 9 "Net-(BT1-Pad2)"))
+    (model ${KISYS3DMOD}/Pin_Headers.3dshapes/Pin_Header_Straight_1x04_Pitch2.54mm.wrl
+      (at (xyz 0 0 0))
+      (scale (xyz 1 1 1))
+      (rotate (xyz 0 0 0))
+    )
+  )
+  (module Pin_Headers:Pin_Header_Straight_1x04_Pitch2.54mm (layer F.Cu)
+    (at 134.62 101.6 270)
+    (descr "Through hole straight pin header, 1x04, 2.54mm pitch, single row")
+    (tags "Through hole pin header THT 1x04 2.54mm single row")
+    (fp_text reference J2 (at 0 -2.33 270) (layer F.SilkS)
+      (effects (font (size 1 1) (thickness 0.15)))
+    )
+    (fp_text value Conn_01x04 (at 0 9.95 270) (layer F.Fab)
+      (effects (font (size 1 1) (thickness 0.15)))
+    )
+    (fp_line (start -0.635 -1.27) (end 1.27 -1.27) (layer F.Fab) (width 0.1))
+    (fp_line (start 1.27 -1.27) (end 1.27 8.89) (layer F.Fab) (width 0.1))
+    (fp_line (start 1.27 8.89) (end -1.27 8.89) (layer F.Fab) (width 0.1))
+    (fp_line (start -1.27 8.89) (end -1.27 -0.635) (layer F.Fab) (width 0.1))
+    (fp_line (start -1.27 -0.635) (end -0.635 -1.27) (layer F.Fab) (width 0.1))
+    (fp_line (start -1.33 8.95) (end 1.33 8.95) (layer F.SilkS) (width 0.12))
+    (fp_line (start -1.33 1.27) (end -1.33 8.95) (layer F.SilkS) (width 0.12))
+    (fp_line (start 1.33 1.27) (end 1.33 8.95) (layer F.SilkS) (width 0.12))
+    (fp_line (start -1.33 1.27) (end 1.33 1.27) (layer F.SilkS) (width 0.12))
+    (fp_line (start -1.33 0) (end -1.33 -1.33) (layer F.SilkS) (width 0.12))
+    (fp_line (start -1.33 -1.33) (end 0 -1.33) (layer F.SilkS) (width 0.12))
+    (fp_line (start -1.8 -1.8) (end -1.8 9.4) (layer F.CrtYd) (width 0.05))
+    (fp_line (start -1.8 9.4) (end 1.8 9.4) (layer F.CrtYd) (width 0.05))
+    (fp_line (start 1.8 9.4) (end 1.8 -1.8) (layer F.CrtYd) (width 0.05))
+    (fp_line (start 1.8 -1.8) (end -1.8 -1.8) (layer F.CrtYd) (width 0.05))
+    (fp_text user %R (at 0 3.81 360) (layer F.Fab)
+      (effects (font (size 1 1) (thickness 0.15)))
+    )
+    (pad 1 thru_hole rect (at 0 0 270) (size 1.7 1.7) (drill 1) (layers *.Cu *.Mask)
+      (net 7 "Net-(BT1-Pad1)"))
+    (pad 2 thru_hole oval (at 0 2.54 270) (size 1.7 1.7) (drill 1) (layers *.Cu *.Mask)
+      (net 3 "Net-(D1-Pad2)"))
+    (pad 3 thru_hole oval (at 0 5.08 270) (size 1.7 1.7) (drill 1) (layers *.Cu *.Mask)
+      (net 15 "Net-(J2-Pad3)"))
+    (pad 4 thru_hole oval (at 0 7.62 270) (size 1.7 1.7) (drill 1) (layers *.Cu *.Mask)
+      (net 2 "Net-(C1-Pad2)"))
+    (model ${KISYS3DMOD}/Pin_Headers.3dshapes/Pin_Header_Straight_1x04_Pitch2.54mm.wrl
       (at (xyz 0 0 0))
       (scale (xyz 1 1 1))
@@
   (segment (start 132.08 113.35) (end 130.175 113.35) (width 0.25) (layer F.Cu) (net 11))
   (segment (start 130.175 113.35) (end 129.855 113.03) (width 0.25) (layer F.Cu) (net 11))
-  (segment (start 122.87 118.745) (end 122.87 117.475) (width 0.25) (layer F.Cu) (net 12))
-  (segment (start 122.87 117.475) (end 123.19 117.155) (width 0.25) (layer F.Cu) (net 12))
-  (segment (start 139.7 113.03) (end 139.7 111.76) (width 0.25) (layer F.Cu) (net 13))
-  (segment (start 138.43 110.49) (end 135.94 110.49) (width 0.25) (layer F.Cu) (net 13))
-  (segment (start 139.7 111.76) (end 138.43 110.49) (width 0.25) (layer F.Cu) (net 13))
-  (segment (start 135.94 110.49) (end 135.62 110.17) (width 0.25) (layer F.Cu) (net 13))
-  (segment (start 139.7 113.03) (end 139.7 117.16) (width 0.25) (layer F.Cu) (net 13))
-  (segment (start 139.7 113.03) (end 139.7 113.03) (width 0.25) (layer F.Cu) (net 13))
+  (segment (start 139.7 113.03) (end 139.7 111.76) (width 0.25) (layer F.Cu) (net 12))
+  (segment (start 138.43 110.49) (end 135.94 110.49) (width 0.25) (layer F.Cu) (net 12))
+  (segment (start 139.7 111.76) (end 138.43 110.49) (width 0.25) (layer F.Cu) (net 12))
+  (segment (start 135.94 110.49) (end 135.62 110.17) (width 0.25) (layer F.Cu) (net 12))
+  (segment (start 139.7 113.03) (end 139.7 117.16) (width 0.25) (layer F.Cu) (net 12))
+  (segment (start 139.7 113.03) (end 139.7 113.03) (width 0.25) (layer F.Cu) (net 12))
+  (segment (start 122.87 118.745) (end 122.87 117.475) (width 0.25) (layer F.Cu) (net 13))
+  (segment (start 122.87 117.475) (end 123.19 117.155) (width 0.25) (layer F.Cu) (net 13))
 )

Commit message: new footprint
switched to offset smd
in correct position to match DIP
Parts:
- J1, J2: footprint Pin_Headers:Pin_Header_Straight_1x04_Pitch2.54mm -> Pin_Headers:Pin_Header_Straight_1x04_Pitch2.54mm_SMD_Pin1Right; moved to B.Cu
- moved J1 15.9 mm to (134.6, 113.0), turned to 0 degrees
- moved J2 13.7 mm to (127.0, 113.0), turned to 180 degrees
Other:
- net class Default: clearance 0.2 -> 0.25
- rule trace_clearance: 0.2 -> 0.25

Commit message: replace BC8*7 with MMBT390* transistors
Parts:
- Q1, Q3, Q4: value BC847 -> MMBT3904
- Q2A1, Q2B1: value BC807 -> MMBT3906
Changed lines of the file:
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@@
     (links 32)
     (no_connects 6)
-    (area 108.232381 105.695 150.84762 121.735)
+    (area 0 0 0 0)
     (thickness 1.6)
     (drawings 0)
@@
       (effects (font (size 1 1) (thickness 0.15)))
     )
-    (fp_text value BC847 (at 0 2.5) (layer F.Fab)
+    (fp_text value MMBT3904 (at 0 2.5) (layer F.Fab)
       (effects (font (size 1 1) (thickness 0.15)))
     )
@@
       (effects (font (size 1 1) (thickness 0.15)))
     )
-    (fp_text value BC807 (at 0 2.5) (layer F.Fab)
+    (fp_text value MMBT3906 (at 0 2.5) (layer F.Fab)
       (effects (font (size 1 1) (thickness 0.15)))
     )
@@
       (effects (font (size 1 1) (thickness 0.15)))
     )
-    (fp_text value BC807 (at 0 2.5) (layer F.Fab)
+    (fp_text value MMBT3906 (at 0 2.5) (layer F.Fab)
       (effects (font (size 1 1) (thickness 0.15)))
     )
@@
       (effects (font (size 1 1) (thickness 0.15)))
     )
-    (fp_text value BC847 (at 0 2.5 180) (layer F.Fab)
+    (fp_text value MMBT3904 (at 0 2.5 180) (layer F.Fab)
       (effects (font (size 1 1) (thickness 0.15)))
     )
@@
       (effects (font (size 1 1) (thickness 0.15)))
     )
-    (fp_text value BC847 (at 0 2.5 270) (layer F.Fab)
-      (effects (font (size 1 1) (thickness 0.15)))
-    )
+    (fp_text value MMBT3904 (at 0 2.5 270) (layer F.Fab)
+      (effects (font (size 1 1) (thickness 0.15)))
+    )
