File: LM3909.sch (KiCad schematic (older format))
At the start: 20 parts, among them J1 Conn_01x04, J2 Conn_01x04, Q1 MMBT3904, Q2A1 MMBT3906, Q2B1 MMBT3906, Q3 MMBT3904, Q4 MMBT3904

Commit message: increase cap footprint to 0805
Parts:
- C1: footprint Capacitors_SMD:C_0805 -> Capacitors_SMD:C_1206
Changed lines of the file:
@@
 F 0 "C1" H 2725 2500 50  0000 L CNN
 F 1 "C" H 2725 2300 50  0000 L CNN
-F 2 "Capacitors_SMD:C_0805" H 2738 2250 50  0001 C CNN
+F 2 "Capacitors_SMD:C_1206" H 2738 2250 50  0001 C CNN
 F 3 "" H 2700 2400 50  0001 C CNN
 	1    2700 2400

Commit message: change resistors from 410 to 510 ohm
Parts:
- R4, R5: value 410 -> 510
Changed lines of the file:
@@
 P 3000 1750
 F 0 "R4" V 3080 1750 50  0000 C CNN
-F 1 "410" V 3000 1750 50  0000 C CNN
+F 1 "510" V 3000 1750 50  0000 C CNN
 F 2 "Resistors_SMD:R_0805" V 2930 1750 50  0001 C CNN
 F 3 "" H 3000 1750 50  0001 C CNN
@@
 P 3000 2150
 F 0 "R5" V 3080 2150 50  0000 C CNN
-F 1 "410" V 3000 2150 50  0000 C CNN
+F 1 "510" V 3000 2150 50  0000 C CNN
 F 2 "Resistors_SMD:R_0805" V 2930 2150 50  0001 C CNN
 F 3 "" H 3000 2150 50  0001 C CNN
